Commit message: add ros ignore and upload robot urdf

File: catkin_ws/src/platform_description/urdf/warthog.urdf.xacro (robot description, xacro)
@@ -298,28 +298,28 @@
     <parent link="imu_link"/>
     <child link="velodyne" />
-    <origin xyz="0.6 0 0" rpy="0 3.1415926 -1.5707463" />
-  </joint>
-  <link name="ouster_frame" />
-  <joint name="ouster_to_imu" type="fixed">
+    <origin xyz="0.6 0 0" rpy="0 3.1415926 -3.1415926" />
+  </joint>
+  <link name="os1_frame" />
+  <joint name="os1_to_imu" type="fixed">
     <parent link="imu_link"/>
-    <child link="ouster_frame" />
+    <child link="os1_frame" />
     <origin xyz="0.45 0 -0.07" rpy="0 3.1415926 0" />
   </joint>
-  <link name="ouster_sensor" />
-  <joint name="ouster_sensor_to_ouster_frame" type="fixed">
-    <parent link="ouster_frame"/>
-    <child link="ouster_sensor" />
+  <link name="os1_sensor" />
+  <joint name="os1_sensor_to_os1_frame" type="fixed">
+    <parent link="os1_frame"/>
+    <child link="os1_sensor" />
     <origin xyz="0 0 0" rpy="0 0 -3.1415926" />
   </joint>
-  <link name="ouster_lidar" />
-  <joint name="ouster_lidar_to_ouster_sensor" type="fixed">
-    <parent link="ouster_sensor"/>
-    <child link="ouster_lidar" />
+  <link name="os1_lidar" />
+  <joint name="os1_lidar_to_os1_sensor" type="fixed">
+    <parent link="os1_sensor"/>
+    <child link="os1_lidar" />
     <origin xyz="0 0 0.03618" rpy="0 0 -3.1415927" />
   </joint>
-  <link name="ouster_imu" />
-  <joint name="ouster_imu_to_ouster_sensor" type="fixed">
-    <parent link="ouster_sensor"/>
-    <child link="ouster_imu" />
+  <link name="os1_imu" />
+  <joint name="os1_imu_to_os1_sensor" type="fixed">
+    <parent link="os1_sensor"/>
+    <child link="os1_imu" />
     <origin xyz="0.006253 -0.011775 0.007645" rpy="0 0 0" />
   </joint>
